File: Minilab/Minilab.kicad_sch (KiCad schematic)
At the start: 53 parts, among them J1 Salida, J2 Screw_Terminal_01x03, J3 Entradas, J4 Salidas, J5 Oscilador, J6 USB_C_Receptacle_USB2.0_14P, J7 DIN41612_02x16_AB, SW1 SW_2, SW2 SW_DIP_x06, U1 4049, U2 NE555D, U78 LM7805_TO220

Commit message: Actualizacion3
Parts:
- J6: now left out of the parts list
Connections:
- net 5V: no longer R3.1, U1.1 (VCC), U2.4 (~{RST}), U2.8 (VCC)
- net GND: no longer BT1.2 (-), C10.2, C11.2, C3.2, J1.2 (Pin_2), J2.1 (Pin_1), J6.A1 (GND), J6.A12 (GND), J6.B1 (GND), J6.B12 (GND), J6.SH (SHIELD), R1.2, R4.2, U2.1 (GND), U78.2 (GND)
- new net: R3.1, U2.4 (~{RST}), U2.8 (VCC)
- new net GND 1: BT1.2 (-), C10.2, C11.2, J1.2 (Pin_2), J2.1 (Pin_1), J6.A1 (GND), J6.A12 (GND), J6.B1 (GND), J6.B12 (GND), J6.SH (SHIELD), R1.2, U78.2 (GND)
- new net GND 2: C3.2, R4.2, U2.1 (GND)
Changed lines of the file:
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@@
 	)
 	(junction
-		(at 99.06 35.56)
+		(at 99.06 38.1)
 		(diameter 0)
 		(color 0 0 0 0)
@@
 	)
 	(junction
-		(at 210.82 110.49)
-		(diameter 0)
-		(color 0 0 0 0)
-	)
-	(junction
 		(at 124.46 67.31)
 		(diameter 0)
@@
 	(wire
 		(pts
-			(xy 99.06 35.56) (xy 99.06 41.91)
+			(xy 99.06 35.56) (xy 99.06 38.1)
 		)
 		(stroke
@@
 	(wire
 		(pts
+			(xy 99.06 38.1) (xy 99.06 41.91)
+		)
+		(stroke
+			(width 0)
+			(type default)
+		)
+	)
+	(wire
+		(pts
 			(xy 213.36 102.87) (xy 213.36 100.33)
 		)
@@
 	(wire
 		(pts
-			(xy 210.82 110.49) (xy 210.82 115.57)
-		)
-		(stroke
-			(width 0)
-			(type default)
-		)
-	)
-	(wire
-		(pts
 			(xy 78.74 110.49) (xy 91.44 110.49)
 		)
@@
 	(wire
 		(pts
-			(xy 99.06 35.56) (xy 101.6 35.56)
-		)
-		(stroke
-			(width 0)
-			(type default)
-		)
-	)
-	(wire
-		(pts
 			(xy 213.36 50.8) (xy 213.36 49.53)
 		)
@@
 	(wire
 		(pts
+			(xy 99.06 38.1) (xy 101.6 38.1)
+		)
+		(stroke
+			(width 0)
+			(type default)
+		)
+	)
+	(wire
+		(pts
 			(xy 144.78 64.77) (xy 158.75 64.77)
 		)
@@
 		)
 	)
-	(global_label "5V USB"
-		(shape input)
-		(at 33.02 91.44 180)
-		(fields_autoplaced yes)
-		(effects
-			(font
-				(size 1.27 1.27)
-			)
-			(justify right)
-		)
-		(property "Intersheetrefs" "${INTERSHEET_REFS}"
-			(at 22.9591 91.44 0)
-			(hide yes)
-			(show_name no)
-			(do_not_autoplace no)
-			(effects
-				(font
-					(size 1.27 1.27)
-				)
-				(justify right)
-			)
-		)
-	)
 	(global_label "S2"
 		(shape input)
@@
 		)
 	)
-	(global_label "5V"
-		(shape input)
-		(at 101.6 35.56 0)
-		(fields_autoplaced yes)
-		(effects
-			(font
-				(size 1.27 1.27)
-			)
-			(justify left)
-		)
-		(property "Intersheetrefs" "${INTERSHEET_REFS}"
-			(at 106.8833 35.56 0)
-			(hide yes)
-			(show_name no)
-			(do_not_autoplace no)
-			(effects
-				(font
-					(size 1.27 1.27)
-				)
-				(justify left)
-			)
-		)
-	)
 	(global_label "E3"
 		(shape input)
@@
 		)
 	)
-	(global_label "5V"
+	(global_label "E5"
 		(shape input)
-		(at 33.02 95.25 180)
+		(at 260.35 120.65 0)
 		(fields_autoplaced yes)
 		(effects
@@
 				(size 1.27 1.27)
 			)
-			(justify right)
+			(justify left)
 		)
 		(property "Intersheetrefs" "${INTERSHEET_REFS}"
-			(at 27.7367 95.25 0)
+			(at 265.6937 120.65 0)
 			(hide yes)
 			(show_name no)
@@
 					(size 1.27 1.27)
 				)
-				(justify right)
+				(justify left)
 			)
 		)
 	)
-	(global_label "E5"
+	(global_label "5V USB"
 		(shape input)
-		(at 260.35 120.65 0)
+		(at 101.6 38.1 0)
 		(fields_autoplaced yes)
 		(effects
@@
 		)
 		(property "Intersheetrefs" "${INTERSHEET_REFS}"
-			(at 265.6937 120.65 0)
+			(at 111.6609 38.1 0)
 			(hide yes)
 			(show_name no)
@@
 		)
 	)
-	(global_label "5V"
-		(shape input)
-		(at 210.82 110.49 180)
-		(fields_autoplaced yes)
-		(effects
-			(font
-				(size 1.27 1.27)
-			)
-			(justify right)
-		)
-		(property "Intersheetrefs" "${INTERSHEET_REFS}"
-			(at 205.5367 110.49 0)
-			(hide yes)
-			(show_name no)
-			(do_not_autoplace no)
-			(effects
-				(font
-					(size 1.27 1.27)
-				)
-				(justify right)
-			)
-		)
-	)
 	(global_label "E5"
 		(shape input)
@@
 		)
 	)
-	(global_label "5V USB"
-		(shape input)
-		(at 210.82 115.57 180)
-		(fields_autoplaced yes)
-		(effects
-			(font
-				(size 1.27 1.27)
-			)
-			(justify right)
-		)
-		(property "Intersheetrefs" "${INTERSHEET_REFS}"
-			(at 200.7591 115.57 0)
-			(hide yes)
-			(show_name no)
-			(do_not_autoplace no)
-			(effects
-				(font
-					(size 1.27 1.27)
-				)
-				(justify right)
-			)
-		)
-	)
 	(global_label "S4"
 		(shape input)
@@
 			)
 		)
-		(property "Value" "GND"
+		(property "Value" "GND 1"
 			(at 38.1 193.04 0)
 			(show_name no)
@@
 			)
 		)
-		(property "Value" "GND"
+		(property "Value" "GND 1"
 			(at 60.96 58.42 0)
 			(show_name no)
@@
 		(body_style 1)
 		(exclude_from_sim no)
-		(in_bom yes)
-		(on_board yes)
+		(in_bom no)
+		(on_board no)
 		(in_pos_files yes)
 		(dnp no)
@@
 			)
 		)
-		(property "Value" "GND"
+		(property "Value" "GND 2"
 			(at 41.91 133.35 0)
 			(show_name no)
@@
 					(unit 1)
 				)
+			)
+		)
+	)
+	(symbol
+		(lib_id "power:PWR_FLAG")
+		(at 33.02 91.44 0)
+		(unit 1)
+		(body_style 1)
+		(exclude_from_sim no)
+		(in_bom yes)
+		(on_board yes)
+		(in_pos_files yes)
+		(dnp no)
+		(property "Reference" "#FLG05"
+			(at 33.02 89.535 0)
+			(hide yes)
+			(show_name no)
+			(do_not_autoplace no)
+			(effects
+				(font
+					(size 1.27 1.27)
+				)
+			)
+		)
+		(property "Value" "PWR_FLAG"
+			(at 33.02 86.614 0)
+			(show_name no)
+			(do_not_autoplace no)
+			(effects
+				(font
+					(size 1.27 1.27)
+				)
+			)
+		)
+		(property "Footprint" ""
+			(at 33.02 91.44 0)
+			(hide yes)
+			(show_name no)
+			(do_not_autoplace no)
+			(effects
+				(font
+					(size 1.27 1.27)
+				)
+			)
+		)
+		(property "Datasheet" ""
+			(at 33.02 91.44 0)
+			(hide yes)
+			(show_name no)
+			(do_not_autoplace no)
+			(effects
+				(font
+					(size 1.27 1.27)
+				)
+			)
+		)
+		(property "Description" "Special symbol for telling ERC where power comes from"
+			(at 33.02 91.44 0)
+			(hide yes)
+			(show_name no)
+			(do_not_autoplace no)
+			(effects
+				(font
+					(size 1.27 1.27)
+				)
+			)
+		)
+		(pin "1"
+		)
+		(instances
+			(project "Minilab"
+				(path "/42f973db-d6e2-440d-9388-60b5f6dca35f"
+					(reference "#FLG05")
+					(unit 1)
+				)
